File: pcb/_autosave-stm32-linux-blinkenlights.kicad_pcb (KiCad board)
At the start: 2 copper layers, 70 x 50 mm, 42 parts, among them J1 USB_C_Receptacle, J2 Conn_01x04_Socket, SW1 SW_Push, U1 LM2575-3.3BT, U2 STM32F103C8Tx

Commit message: update pcb
Signed-off-by: Nia Schlegel <gott@3nt3.de>
Parts:
- C3: value C -> 100n
- C4, C5, C6, C7: value 100u -> 100n
Changed lines of the file:
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@@
 			)
 		)
-		(property "Value" "100u"
+		(property "Value" "100n"
 			(at 0 1.43 0)
 			(layer "F.Fab")
@@
 			)
 		)
-		(property "Value" "C"
+		(property "Value" "100n"
 			(at 0 1.43 0)
 			(layer "F.Fab")
@@
 			)
 		)
-		(property "Value" "100u"
+		(property "Value" "100n"
 			(at 0 1.43 0)
 			(layer "F.Fab")
@@
 			)
 		)
-		(property "Value" "100u"
+		(property "Value" "100n"
 			(at 0 1.43 0)
 			(layer "F.Fab")
@@
 			)
 		)
-		(property "Value" "100u"
+		(property "Value" "100n"
 			(at 0 1.43 0)
 			(layer "F.Fab")
