File: pcb/stm32-linux-blinkenlights.kicad_sch (KiCad schematic)
At the start: 38 parts, among them J2 Conn_01x04_Socket, J3 USB_C_Receptacle, SW1 SW_Push, U1 STM32F103C8Tx, U2 LM2575-3.3BT

Commit message: update pcb
Signed-off-by: Nia Schlegel <gott@3nt3.de>
Parts:
- removed C4, C7: 100u, Capacitor_SMD:C_0603_1608Metric_Pad1.08x0.95mm_HandSolder, symbol Device:C
- added C1: 100u, Capacitor_SMD:CP_Elec_6.3x7.7, symbol Device:C_Polarized
- C3: renamed from C6; value C -> 100n
- C4: renamed from C1; value 100u -> 100n
- C5: renamed from C2; value 100u -> 100n
- C6: renamed from C3; value 100u -> 100n
- C7: renamed from C5; value 100u -> 100n
- D1: renamed from D11; footprint Diode_THT:D_DO-41_SOD81_P10.16mm_Horizontal -> Diode_SMD:D_SOD-123
- J1: renamed from J3; footprint (none) -> easyeda2kicad:USB-C-SMD_TYPE-C-6PIN-2MD-073
- R1: renamed from R12; footprint LED_SMD:LED_0603_1608Metric_Pad1.05x0.95mm_HandSolder -> Resistor_SMD:R_0603_1608Metric_Pad0.98x0.95mm_HandSolder
- R10: renamed from R7; footprint LED_SMD:LED_0603_1608Metric_Pad1.05x0.95mm_HandSolder -> Resistor_SMD:R_0603_1608Metric_Pad0.98x0.95mm_HandSolder
- R11: renamed from R8; footprint LED_SMD:LED_0603_1608Metric_Pad1.05x0.95mm_HandSolder -> Resistor_SMD:R_0603_1608Metric_Pad0.98x0.95mm_HandSolder
- R12: renamed from R9; footprint LED_SMD:LED_0603_1608Metric_Pad1.05x0.95mm_HandSolder -> Resistor_SMD:R_0603_1608Metric_Pad0.98x0.95mm_HandSolder
- R13: renamed from R10; footprint LED_SMD:LED_0603_1608Metric_Pad1.05x0.95mm_HandSolder -> Resistor_SMD:R_0603_1608Metric_Pad0.98x0.95mm_HandSolder
- R2: renamed from R13; footprint LED_SMD:LED_0603_1608Metric_Pad1.05x0.95mm_HandSolder -> Resistor_SMD:R_0603_1608Metric_Pad0.98x0.95mm_HandSolder
- R3: renamed from R11; footprint LED_SMD:LED_0603_1608Metric_Pad1.05x0.95mm_HandSolder -> Resistor_SMD:R_0603_1608Metric_Pad0.98x0.95mm_HandSolder
- R4: renamed from R1; footprint LED_SMD:LED_0603_1608Metric_Pad1.05x0.95mm_HandSolder -> Resistor_SMD:R_0603_1608Metric_Pad0.98x0.95mm_HandSolder
- R5: renamed from R2; footprint LED_SMD:LED_0603_1608Metric_Pad1.05x0.95mm_HandSolder -> Resistor_SMD:R_0603_1608Metric_Pad0.98x0.95mm_HandSolder
- R6: renamed from R3; footprint LED_SMD:LED_0603_1608Metric_Pad1.05x0.95mm_HandSolder -> Resistor_SMD:R_0603_1608Metric_Pad0.98x0.95mm_HandSolder
- R7: renamed from R4; footprint LED_SMD:LED_0603_1608Metric_Pad1.05x0.95mm_HandSolder -> Resistor_SMD:R_0603_1608Metric_Pad0.98x0.95mm_HandSolder
- R8: renamed from R5; footprint LED_SMD:LED_0603_1608Metric_Pad1.05x0.95mm_HandSolder -> Resistor_SMD:R_0603_1608Metric_Pad0.98x0.95mm_HandSolder
- R9: renamed from R6; footprint LED_SMD:LED_0603_1608Metric_Pad1.05x0.95mm_HandSolder -> Resistor_SMD:R_0603_1608Metric_Pad0.98x0.95mm_HandSolder
- renumbered C8 to C2, D9 to D10, D10 to D11, D1 to D2, D2 to D3, D3 to D4, D4 to D5, D5 to D6, D6 to D7, D7 to D8, D8 to D9, U2 to U1, U1 to U2
Connections:
- net VBUS: now also C1.1
- net at C2.2, D1.2 (A), U1.3 (GND): now also U1.5 (~{ON}/OFF), C1.2
Other:
- moved on the sheet: C7

Commit message: v0.2?
Signed-off-by: Nia Schlegel <gott@3nt3.de>
Parts:
- removed C1: 100u, Capacitor_SMD:CP_Elec_6.3x7.7, symbol Device:C_Polarized
- removed C2: 330u, Capacitor_SMD:CP_Elec_6.3x7.7, symbol Device:C_Polarized
- removed D1: 1N5819, Diode_SMD:D_SOD-123, symbol Diode:1N5819
- removed L1: 330u, Inductor_SMD:L_6.3x6.3_H3, symbol Device:L
- removed U1: LM2575-3.3BT, Package_TO_SOT_SMD:TO-263-5_TabPin6, symbol Regulator_Switching:LM2575-3.3BT
- added C1, C10, C2: 100n, Capacitor_SMD:C_0603_1608Metric_Pad1.08x0.95mm_HandSolder, symbol Device:C
- added C4, C8: 10p, Capacitor_SMD:C_0603_1608Metric_Pad1.08x0.95mm_HandSolder, symbol Device:C
- added H1, H2, H3, H4: MountingHole, MountingHole:MountingHole_3.5mm_Pad, symbol Mechanical:MountingHole
- added U1: LP5907MFX-3.3, Package_TO_SOT_SMD:SOT-23-5, symbol Regulator_Linear:LP5907MFX-3.3
- added Y1: Crystal_GND24, Crystal:Crystal_SMD_3225-4Pin_3.2x2.5mm_HandSoldering, symbol Device:Crystal_GND24
- C3: renamed from C4; footprint LED_SMD:LED_0603_1608Metric_Pad1.05x0.95mm_HandSolder -> Capacitor_SMD:C_0603_1608Metric_Pad1.08x0.95mm_HandSolder
- J1: footprint easyeda2kicad:USB-C-SMD_TYPE-C-6PIN-2MD-073 -> easyeda2kicad:USB-C-SMD_MC-311D
- R10, R11, R12, R13, R4, R5, R6, R7, R8, R9: value 47R -> 680R
- renumbered C3 to C6, C6 to C7, C7 to C9, D2 to D1, D11 to D10, D3 to D2, D4 to D3, D5 to D4, D6 to D5, D7 to D6, D8 to D7, D9 to D8, D10 to D9
Connections:
- net +3.3V: now also C10.1, C2.1, U1.5 (OUT)
- net GND: now also C1.2, C10.2, C2.2, C4.2, C8.2, U1.2 (GND), Y1.2, Y1.4; no longer D1.1 (K), D10.1 (K), D2.1 (K), D3.1 (K), D4.1 (K), D5.1 (K), D6.1 (K), D7.1 (K), D8.1 (K), D9.1 (K), J1.S1 (SHIELD)
- net VBUS: now also D1.2 (A), D10.2 (A), D2.2 (A), D3.2 (A), D4.2 (A), D5.2 (A), D6.2 (A), D7.2 (A), D8.2 (A), D9.2 (A), C1.1, U1.1 (IN), U1.3 (EN)
- net at R7.1: now also D4.1 (K); no longer D4.2 (A)
- net at R13.1: now also D10.1 (K); no longer D10.2 (A)
- net at R10.1: now also D7.1 (K); no longer D7.2 (A)
- net at R9.1: now also D6.1 (K); no longer D6.2 (A)
- net at R11.1: now also D8.1 (K); no longer D8.2 (A)
- net at R5.1: now also D2.1 (K); no longer D2.2 (A)
- net at R8.1: now also D5.1 (K); no longer D5.2 (A)
- net at R4.1: now also D1.1 (K); no longer D1.2 (A)
- net at R6.1: now also D3.1 (K); no longer D3.2 (A)
- net at R12.1: now also D9.1 (K); no longer D9.2 (A)
- net at U2.5 (PD0): now also C4.1, Y1.1
- net at U2.6 (PD1): now also C8.1, Y1.3
- net SWCLK: no longer names the net of J2.2 (Pin_2)
- net SWCLK: now also U2.34 (PA13); no longer U2.37 (PA14)
- net SWDIO: no longer names the net of J2.3 (Pin_3)
- net SWDIO: now also U2.37 (PA14); no longer U2.34 (PA13)
- no-connect marks 33 -> 32
Other:
- note added: "LED Array"
- note added: "Power"
- note added: "USB"
- moved on the sheet: C3, C5, C6, C7, C9, D1, D10, D2, D3, D4, D5, D6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
